File: Hardware/V3/Pi Zero PITS.brd (EAGLE design)
At the start: 100.2 x 29.9 mm, 43 parts, among them IC1 MCP3426_ignore pin names, U1 U1, U2 LORA, U3 DS18B20, U4 MAX40200AUK+21-0057F_MXM-M

Commit message: Printed
Parts:
- removed GREEN: (no value), led:SML0603
- removed PAD2: (no value), KEW_HF_V13:SMD_SMALL
- removed R4, R5: 330 0603, rcl:R0603
- removed U$2: MIC9409X_MIC9409X, KEW_HF_V13:MIC9409X_DCK_R-PDSO-G6
- removed U$3: SOLARPAD, KEW_HF_V13:SOLARMOUNT
- added C11, C12, C13: 100nF 0603, rcl:C0603K
- added GRN: (no value), led:SML0603
- added PAD4, PAD5, S+: (no value), KEW_HF_V13:SMD_SMALL
- added R4R, R5G: 330 0603, rcl:R0603
- added RB2, RB3: 0 0603, rcl:R0603
- added S-: S-, KEW_HF_V13:SMD_SMALL
- added U5: MAX40200AUK+21-0057F_MXM-M, KEW_HF_V13:21-0057F_MXM-M
- moved U4 19.0 mm to (42.5, 17.8), turned to 180 degrees
- moved RED 18.5 mm to (82.5, 14.6)
- moved C7 17.1 mm to (57.4, 30.9), flipped to the top, turned to 270 degrees
- moved R1 16.3 mm to (28.2, 13.7), turned to 90 degrees
- moved C8 12.8 mm to (75.6, 28.6), turned to 90 degrees
- moved C6 11.8 mm to (55.9, 24.6), flipped to the top, turned to 90 degrees
- moved R2 10.8 mm to (50.8, 24.6), flipped to the top, turned to 270 degrees
- moved C9 10.7 mm to (75.6, 24.8), turned to 90 degrees
- moved C1 8.79 mm to (35.6, 29.8), flipped to the top, turned to 270 degrees
- moved R3 8.03 mm to (53.3, 24.6), flipped to the top, turned to 90 degrees
- moved C5 7.93 mm to (36.2, 24.5)
- moved C3 7.77 mm to (32.4, 22.9), turned to 0 degrees
- moved CK1 7.18 mm to (32.4, 25.4)
- moved U$4 6.93 mm to (43.8, 24.8), turned to 270 degrees
- moved C4 6.09 mm to (32.4, 27.9), turned to 0 degrees
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- renumbered R7 to RB1
Connections:
- removed net NSS: CH_SEL.2, U2.P$13
- removed net VDD: U4.1
- new net N$18: C11.1, RB1.1, RB2.2, SW1.3, SW1.4, U5.1, U5.3
- new net N$19: C13.1, RB3.2, S+.1, U4.1, U4.3
- net 3V3#1: now also R1.1, U$4.VCC, U3.3; no longer C7.1, IC1.3
- net 3V3#2: now also C7.1, IC1.3; no longer R1.1, U$4.VCC, U3.3
- net 5V_IN: now also C12.1, RB2.1, RB3.1, U4.5, U5.5; no longer RB1.1, SW1.3, SW1.4
- net CS0: now also CH_SEL.2, U2.P$13
- net GND: now also C11.2, C12.2, C13.2, R4R.1, R5G.1, S-.1, U4.2, U5.2; no longer R4.1, R5.1
- net LED2: now also GRN.A; no longer GREEN.A
- net N$3: now also GRN.C, R5G.2; no longer GREEN.C, R5.2
- net N$8: now also R4R.2; no longer R4.2
Routing:
- net DQ: track 0.00 -> 43.4 mm, vias 0 -> 2
- net 3V3#1: track 14.1 -> 53.0 mm, vias 0 -> 3
- net 5V_IN: track 20.0 -> 57.6 mm, vias 0 -> 3
- net GPS_TX/PI_RX: track 0.00 -> 34.8 mm, vias 0 -> 1
- net CS0: track 6.36 -> 38.6 mm, vias 0 -> 3
- net GPS_RX/PI_TX: track 0.00 -> 31.4 mm, vias 0 -> 1
- net NSS: track 26.6 -> 0.00 mm, vias 1 -> 0
- net N$18: track 0.00 -> 23.0 mm
- net 3V3#2: track 36.1 -> 55.5 mm, vias 0 -> 3
- net LED1: track 3.20 -> 21.0 mm, vias 0 -> 1
- net LED2: track 3.84 -> 21.2 mm, vias 0 -> 1
- net BUTTON: track 0.03 -> 15.9 mm
- net SDA: track 0.03 -> 14.9 mm, vias 0 -> 1
- net N$19: track 0.00 -> 14.8 mm, vias 0 -> 2
- net SCK: track 36.5 -> 26.6 mm
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Other:
- board text added: "If Found Please Call Kevin Walton +44 7867 825 847"
- board text added: "JLCJLCJLCJLC"
- board text added: "PI Zero PITS V3"
