File: Hardware/V4/Pi Zero PITS.sch (EAGLE design)
At the start: 51 parts, among them IC1 MCP3426_ignore pin names, U1 U1, U2 LORA, U3 DS18B20, U4 MAX40200AUK+21-0057F_MXM-M, U5 MAX40200AUK+21-0057F_MXM-M

Commit message: Printed
Parts:
- removed S-1: S-, KEW_HF_V13:SMD2SMD_KW
- removed U3: DS18B20, SparkFun-Sensors:DS18B20
- added U6: DS18B20, DS18B20:DS18B20
- S-: value SOLARPAD -> S-; device KEW_HF_V13:SOLARPAD -> KEW_HF_V13:SMD2SMD_KW
- renumbered R4 to RB2, R5 to RB3, R7 to RB1
Connections:
- removed net N$1: +.1, RB1.2, SW1.1, SW1.2
- removed net N$18: C11.1, RB1.1, RB2.2, SW1.3, SW1.4, U5.EN, U5.VDD
- removed net NSS: CH_SEL.2, U2.P$13
- net 3V3#1: now also R1.1, U$4.VCC, U6.VDD; no longer C7.1, IC1.GND
- net 3V3#2: now also C7.1, IC1.GND; no longer R1.1, U$4.VCC, U3.VDD
- net 5V_IN: now also +.1, C11.1, RB1.1, RB1.2, RB2.2, SW1.2, SW1.3, U5.EN, U5.VDD
- net CS0: now also CH_SEL.2, U2.P$13
- net DQ: now also U6.DQ; no longer U3.DQ
- net GND: now also SW1.1, SW1.4, U6.GND; no longer S-1.P, U3.GND
Other:
- moved on the sheet: +, C11, SW1

Commit message: Added NMEA Logs, minor PCB updates, Git notes and Pi Ethernet Driver
Parts:
- renumbered U$4 to 18B20Z
Changed lines of the file:
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@@
 <part name="GND38" library="SparkFun" deviceset="GND" device=""/>
 <part name="CK1" library="rcl" library_urn="urn:adsk.eagle:library:334" deviceset="R-EU_" device="R0603" package3d_urn="urn:adsk.eagle:package:23555/2" value="BLM18EG601SN1D"/>
-<part name="U$4" library="ava" deviceset="DS1820" device="SOIC"/>
+<part name="18B20Z" library="ava" deviceset="DS1820" device="SOIC"/>
 <part name="CK2" library="rcl" library_urn="urn:adsk.eagle:library:334" deviceset="R-EU_" device="R0402" package3d_urn="urn:adsk.eagle:package:23547/2" value="BLM15HD102SN1D"/>
 <part name="CK3" library="rcl" library_urn="urn:adsk.eagle:library:334" deviceset="R-EU_" device="R0402" package3d_urn="urn:adsk.eagle:package:23547/2" value="BLM15HD102SN1D"/>
@@
 <attribute name="VALUE" x="95.25" y="173.482" size="1.778" layer="96" rot="R180"/>
 </instance>
-<instance part="U$4" gate="G$1" x="246.38" y="63.5" smashed="yes" rot="R270"/>
+<instance part="18B20Z" gate="G$1" x="246.38" y="63.5" smashed="yes" rot="R270"/>
 <instance part="CK2" gate="G$1" x="78.74" y="139.7" smashed="yes">
 <attribute name="NAME" x="69.85" y="141.1986" size="1.778" layer="95"/>
@@
 <segment>
 <pinref part="GND21" gate="1" pin="GND"/>
-<pinref part="U$4" gate="G$1" pin="GND"/>
+<pinref part="18B20Z" gate="G$1" pin="GND"/>
 <wire x1="241.3" y1="68.58" x2="241.3" y2="66.04" width="0.1524" layer="91"/>
 </segment>
@@
 <wire x1="241.3" y1="63.5" x2="233.68" y2="63.5" width="0.1524" layer="91"/>
 <junction x="233.68" y="63.5"/>
-<pinref part="U$4" gate="G$1" pin="DQ"/>
+<pinref part="18B20Z" gate="G$1" pin="DQ"/>
 <wire x1="213.36" y1="63.5" x2="233.68" y2="63.5" width="0.1524" layer="91"/>
 <pinref part="U6" gate="G$1" pin="DQ"/>
@@
 <pinref part="R1" gate="G$1" pin="1"/>
 <wire x1="241.3" y1="60.96" x2="241.3" y2="53.34" width="0.1524" layer="91"/>
-<pinref part="U$4" gate="G$1" pin="VCC"/>
+<pinref part="18B20Z" gate="G$1" pin="VCC"/>
 <wire x1="220.98" y1="58.42" x2="220.98" y2="53.34" width="0.1524" layer="91"/>
 <wire x1="220.98" y1="53.34" x2="233.68" y2="53.34" width="0.1524" layer="91"/>
